File: mariboard.kicad_pcb (KiCad board)
At the start: 2 copper layers, 827 x 356.9 mm, 194 parts, among them U1 ER_OLEDM0.91_1x-I2C, sw1 SW_Push, sw10 SW_Push, sw11 SW_Push, sw12 SW_Push, sw13 SW_Push, sw14 SW_Push, sw15 SW_Push, sw16 SW_Push, sw17 SW_Push, sw18 SW_Push, sw19 SW_Push, sw2 SW_Push, sw20 SW_Push, sw21 SW_Push, sw22 SW_Push, sw23 SW_Push, sw24 SW_Push, sw25 SW_Push, sw26 SW_Push, sw27 SW_Push, sw28 SW_Push, sw29 SW_Push, sw3 SW_Push, sw30 SW_Push, sw31 SW_Push, sw32 SW_Push, sw33 SW_Push, sw34 SW_Push, sw35 SW_Push, sw36 SW_Push, sw37 SW_Push, sw38 SW_Push, sw39 SW_Push, sw4 SW_Push, sw40 SW_Push, sw41 SW_Push, sw42 SW_Push, sw43 SW_Push, sw44 SW_Push, sw45 SW_Push, sw46 SW_Push, sw47 SW_Push, sw48 SW_Push, sw49 SW_Push, sw5 SW_Push, sw50 SW_Push, sw51 SW_Push, sw52 SW_Push, sw53 SW_Push, sw54 SW_Push, sw55 SW_Push, sw56 SW_Push, sw57 SW_Push, sw58 SW_Push, sw59 SW_Push, sw6 SW_Push, sw60 SW_Push, sw61 SW_Push, sw62 SW_Push, sw63 SW_Push, sw64 SW_Push, sw65 SW_Push, sw66 SW_Push, sw67 SW_Push, sw68 SW_Push, sw69 SW_Push, sw7 SW_Push, sw70 SW_Push, sw71 SW_Push, sw72 SW_Push, sw73 SW_Push, sw74 SW_Push, sw75 SW_Push, sw76 SW_Push, sw77 SW_Push, sw78 SW_Push, sw79 SW_Push, sw8 SW_Push, sw80 SW_Push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

Commit message: gerber files update
Parts:
- removed the ? at (555.0, -148.5)
- removed the ? at (498.0, 120.3)
- removed the G*** at (802.8, -37.2)
- removed the G*** at (687.5, -146.8)
- removed the G*** at (813.5, -125.5)
- removed the REF** at (746.1, 54.6)
- removed the REF** at (844.6, -153.6)
- removed the REF** at (479.1, -14.3)
- removed the REF** at (380.6, 193.9)
- removed the REF** at (746.6, 191.6)
- removed the REF** at (845.1, -16.6)
- removed the REF** at (378.6, 54.9)
- removed the REF** at (477.1, -153.3)
- removed the REF** at (746.8, -14.3)
- removed the REF** at (512.1, 194.1)
- removed the REF** at (648.4, 193.9)
- removed the REF** at (610.6, -14.1)
- added ?: LOGO, LOGO, F.Cu at (574.0, -143.4)
- added ?: LOGO, LOGO, B.Cu at (615.1, 125.4)
- added G***: LOGO, LOGO, F.Cu at (832.5, -120.4)
- added G***: LOGO, LOGO, F.Cu at (821.8, -32.2)
- added G***: LOGO, LOGO, F.Cu at (706.5, -141.7)
- added REF**: MountingHole_3.2mm_M3_ISO7380, MountingHole:MountingHole_3.2mm_M3_ISO7380, F.Cu at (497.8, 198.9)
- added REF**: MountingHole_3.2mm_M3_ISO7380, MountingHole:MountingHole_3.2mm_M3_ISO7380, F.Cu at (864.1, -11.5)
- added REF**: MountingHole_3.2mm_M3_ISO7380, MountingHole:MountingHole_3.2mm_M3_ISO7380, F.Cu at (629.2, 199.2)
- added REF**: MountingHole_3.2mm_M3_ISO7380, MountingHole:MountingHole_3.2mm_M3_ISO7380, F.Cu at (863.2, 59.7)
- added REF**: MountingHole_3.2mm_M3_ISO7380, MountingHole:MountingHole_3.2mm_M3_ISO7380, F.Cu at (765.8, -9.27)
- added REF**: MountingHole_3.2mm_M3_ISO7380, MountingHole:MountingHole_3.2mm_M3_ISO7380, F.Cu at (495.8, 59.9)
- added REF**: MountingHole_3.2mm_M3_ISO7380, MountingHole:MountingHole_3.2mm_M3_ISO7380, F.Cu at (496.1, -148.3)
- added REF**: MountingHole_3.2mm_M3_ISO7380, MountingHole:MountingHole_3.2mm_M3_ISO7380, F.Cu at (498.1, -9.27)
- added REF**: MountingHole_3.2mm_M3_ISO7380, MountingHole:MountingHole_3.2mm_M3_ISO7380, F.Cu at (765.5, 198.9)
- added REF**: MountingHole_3.2mm_M3_ISO7380, MountingHole:MountingHole_3.2mm_M3_ISO7380, F.Cu at (629.6, -9.02)
- added REF**: MountingHole_3.2mm_M3_ISO7380, MountingHole:MountingHole_3.2mm_M3_ISO7380, F.Cu at (863.8, 196.7)
- added REF**: MountingHole_3.2mm_M3_ISO7380, MountingHole:MountingHole_3.2mm_M3_ISO7380, F.Cu at (863.6, -148.5)
Other:
- board size 827 x 356.9 mm -> 846 x 357.2 mm

Commit message: Updated Case + BOM
Parts:
- removed the ? at (574.0, -143.4)
- removed the ? at (615.1, 125.4)
- removed the G*** at (832.5, -120.4)
- removed the G*** at (821.8, -32.2)
- removed the G*** at (706.5, -141.7)
- removed the REF** at (497.8, 198.9)
- removed the REF** at (864.1, -11.5)
- removed the REF** at (629.2, 199.2)
- removed the REF** at (863.2, 59.7)
- removed the REF** at (765.8, -9.27)
- removed the REF** at (495.8, 59.9)
- removed the REF** at (496.1, -148.3)
- removed the REF** at (498.1, -9.27)
- removed the REF** at (765.5, 198.9)
- removed the REF** at (629.6, -9.02)
- removed the REF** at (863.8, 196.7)
- removed the REF** at (863.6, -148.5)
- added ?: LOGO, LOGO, F.Cu at (78.5, -144.4)
- added G***: LOGO, LOGO, F.Cu at (365.8, -34.2)
- added G***: LOGO, LOGO, F.Cu at (241.2, -142.1)
Other:
- board size 846 x 357.2 mm -> 382.7 x 148.8 mm
- board text removed: "Keep Out"
- board text removed: "USB Cable"
